Commit message: add new models, improve core_functions

File: eurobot_loc/models/secondary_robot.urdf (robot description, URDF)
Before this commit: robot secondary_robot, 1 links, 0 joints
Links:
- link secondary_robot: geometry visual mesh filename=package://eurobot_loc/models/secondary_robot.STL scale=0.001 0.001 0.001
