Commit message: Refactor useless code

File: eurobot_sim/models/field.urdf (robot description, URDF)
Before this commit: robot field, 2 links, 1 joints
Links:
- link beacons: geometry collision cylinder length=0.1 radius=0.04; collision cylinder length=0.1 radius=0.04
- link table: mass None -> 165.19; geometry visual mesh filename=package://eurobot_sim/models/table.stl.stl

File: eurobot_sim/models/secondary_robot.urdf (robot description, URDF)
Before this commit: robot secondary_robot, 1 links, 0 joints
Links:
- link secondary_robot: geometry visual mesh filename=package://eurobot_loc/models/secondary_robot.STL scale=0.001 0.001 0.001
